File: ILJJ_Mk-V.kicad_pcb (KiCad board)
At the start: 2 copper layers, 48.3 x 99.1 mm, 14 parts, among them J1 Conn_02x12, U1 74LS00, U10 74LS00, U11 74LS00, U2 74LS00, U3 74LS00, U4 74LS00, U5 74LS00, U6 74LS00, U7 74LS00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

Commit message: [add] #1 パワーランプ
抵抗のフットプリントこれでいいのかちょっとあやしい
Parts:
- added D1: POWER, LEDs:LED_D3.0mm, F.Cu at (123.2, 54.0)
- added R1: R, Resistors_ThroughHole:R_Axial_DIN0207_L6.3mm_D2.5mm_P7.62mm_Horizontal, F.Cu at (110.5, 54.0)
Routing:
- net VCC: track 209.2 -> 215.2 mm
- net Net-(D1-Pad2): track 0.00 -> 2.54 mm
Changed lines of the file:
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@@
     (thickness 1.6)
     (drawings 8)
-    (tracks 494)
+    (tracks 498)
     (zones 0)
-    (modules 14)
-    (nets 61)
+    (modules 16)
+    (nets 62)
   )
   (page A4)
@@
   (net 59 "Net-(U11-Pad6)")
   (net 60 "Net-(U11-Pad10)")
+  (net 61 "Net-(D1-Pad2)")
   (net_class Default "これはデフォルトのネット クラスです。"
     (clearance 0.25)
@@
     (add_net /SUB_FLAG)
     (add_net GND)
+    (add_net "Net-(D1-Pad2)")
     (add_net "Net-(J1-Pad13)")
     (add_net "Net-(J1-Pad15)")
@@
     (pad 1 np_thru_hole circle (at 0 0) (size 3 3) (drill 3) (layers *.Cu *.Mask))
   )
+  (module LEDs:LED_D3.0mm (layer F.Cu)
+    (at 123.19 53.975 180)
+    (descr "LED, diameter 3.0mm, 2 pins")
+    (tags "LED diameter 3.0mm 2 pins")
+    (fp_text reference D1 (at 3.81 2.159 180) (layer F.SilkS)
+      (effects (font (size 1 1) (thickness 0.15)))
+    )
+    (fp_text value POWER (at 1.27 2.96 180) (layer F.Fab)
+      (effects (font (size 1 1) (thickness 0.15)))
+    )
+    (fp_line (start 3.7 -2.25) (end -1.15 -2.25) (layer F.CrtYd) (width 0.05))
+    (fp_line (start 3.7 2.25) (end 3.7 -2.25) (layer F.CrtYd) (width 0.05))
+    (fp_line (start -1.15 2.25) (end 3.7 2.25) (layer F.CrtYd) (width 0.05))
+    (fp_line (start -1.15 -2.25) (end -1.15 2.25) (layer F.CrtYd) (width 0.05))
+    (fp_line (start -0.29 1.08) (end -0.29 1.236) (layer F.SilkS) (width 0.12))
+    (fp_line (start -0.29 -1.236) (end -0.29 -1.08) (layer F.SilkS) (width 0.12))
+    (fp_line (start -0.23 -1.16619) (end -0.23 1.16619) (layer F.Fab) (width 0.1))
+    (fp_circle (center 1.27 0) (end 2.77 0) (layer F.Fab) (width 0.1))
+    (fp_arc (start 1.27 0) (end 0.229039 1.08) (angle -87.9) (layer F.SilkS) (width 0.12))
+    (fp_arc (start 1.27 0) (end 0.229039 -1.08) (angle 87.9) (layer F.SilkS) (width 0.12))
+    (fp_arc (start 1.27 0) (end -0.29 1.235516) (angle -108.8) (layer F.SilkS) (width 0.12))
+    (fp_arc (start 1.27 0) (end -0.29 -1.235516) (angle 108.8) (layer F.SilkS) (width 0.12))
+    (fp_arc (start 1.27 0) (end -0.23 -1.16619) (angle 284.3) (layer F.Fab) (width 0.1))
+    (pad 2 thru_hole circle (at 2.54 0 180) (size 1.8 1.8) (drill 0.9) (layers *.Cu *.Mask)
+      (net 61 "Net-(D1-Pad2)"))
+    (pad 1 thru_hole rect (at 0 0 180) (size 1.8 1.8) (drill 0.9) (layers *.Cu *.Mask)
+      (net 7 GND))
+    (model ${KISYS3DMOD}/LEDs.3dshapes/LED_D3.0mm.wrl
+      (at (xyz 0 0 0))
+      (scale (xyz 0.393701 0.393701 0.393701))
+      (rotate (xyz 0 0 0))
+    )
+  )
+  (module Resistors_ThroughHole:R_Axial_DIN0207_L6.3mm_D2.5mm_P7.62mm_Horizontal (layer F.Cu)
+    (at 110.49 53.975)
+    (descr "Resistor, Axial_DIN0207 series, Axial, Horizontal, pin pitch=7.62mm, 0.25W = 1/4W, length*diameter=6.3*2.5mm^2, http://cdn-reichelt.de/documents/datenblatt/B400/1_4W%23YAG.pdf")
+    (tags "Resistor Axial_DIN0207 series Axial Horizontal pin pitch 7.62mm 0.25W = 1/4W length 6.3mm diameter 2.5mm")
+    (fp_text reference R1 (at -1.016 -2.159) (layer F.SilkS)
+      (effects (font (size 1 1) (thickness 0.15)))
+    )
+    (fp_text value R (at 3.81 2.31) (layer F.Fab)
+      (effects (font (size 1 1) (thickness 0.15)))
+    )
+    (fp_line (start 8.7 -1.6) (end -1.05 -1.6) (layer F.CrtYd) (width 0.05))
+    (fp_line (start 8.7 1.6) (end 8.7 -1.6) (layer F.CrtYd) (width 0.05))
+    (fp_line (start -1.05 1.6) (end 8.7 1.6) (layer F.CrtYd) (width 0.05))
+    (fp_line (start -1.05 -1.6) (end -1.05 1.6) (layer F.CrtYd) (width 0.05))
+    (fp_line (start 7.02 1.31) (end 7.02 0.98) (layer F.SilkS) (width 0.12))
+    (fp_line (start 0.6 1.31) (end 7.02 1.31) (layer F.SilkS) (width 0.12))
+    (fp_line (start 0.6 0.98) (end 0.6 1.31) (layer F.SilkS) (width 0.12))
+    (fp_line (start 7.02 -1.31) (end 7.02 -0.98) (layer F.SilkS) (width 0.12))
+    (fp_line (start 0.6 -1.31) (end 7.02 -1.31) (layer F.SilkS) (width 0.12))
+    (fp_line (start 0.6 -0.98) (end 0.6 -1.31) (layer F.SilkS) (width 0.12))
+    (fp_line (start 7.62 0) (end 6.96 0) (layer F.Fab) (width 0.1))
+    (fp_line (start 0 0) (end 0.66 0) (layer F.Fab) (width 0.1))
+    (fp_line (start 6.96 -1.25) (end 0.66 -1.25) (layer F.Fab) (width 0.1))
+    (fp_line (start 6.96 1.25) (end 6.96 -1.25) (layer F.Fab) (width 0.1))
+    (fp_line (start 0.66 1.25) (end 6.96 1.25) (layer F.Fab) (width 0.1))
+    (fp_line (start 0.66 -1.25) (end 0.66 1.25) (layer F.Fab) (width 0.1))
+    (pad 2 thru_hole oval (at 7.62 0) (size 1.6 1.6) (drill 0.8) (layers *.Cu *.Mask)
+      (net 61 "Net-(D1-Pad2)"))
+    (pad 1 thru_hole circle (at 0 0) (size 1.6 1.6) (drill 0.8) (layers *.Cu *.Mask)
+      (net 1 VCC))
+    (model ${KISYS3DMOD}/Resistors_THT.3dshapes/R_Axial_DIN0207_L6.3mm_D2.5mm_P7.62mm_Horizontal.wrl
+      (at (xyz 0 0 0))
+      (scale (xyz 0.393701 0.393701 0.393701))
+      (rotate (xyz 0 0 0))
+    )
+  )
   (gr_line (start 142.24 149.86) (end 109.22 149.86) (layer Edge.Cuts) (width 0.15))
   (gr_line (start 142.24 142.24) (end 142.24 149.86) (layer Edge.Cuts) (width 0.15))
@@
   (segment (start 129.54 59.87) (end 127 62.41) (width 0.25) (layer F.Cu) (net 1))
   (segment (start 127 70.695746) (end 127 71.12001) (width 0.25) (layer F.Cu) (net 1))
+  (segment (start 109.690001 54.774999) (end 110.49 53.975) (width 0.25) (layer F.Cu) (net 1))
+  (segment (start 106.68 57.785) (end 109.690001 54.774999) (width 0.25) (layer F.Cu) (net 1))
+  (segment (start 106.68 58.42) (end 106.68 57.785) (width 0.25) (layer F.Cu) (net 1))
   (segment (start 106.68 131.68) (end 104.14 129.14) (width 0.25) (layer B.Cu) (net 2))
   (segment (start 106.68 132.08) (end 106.68 131.68) (width 0.25) (layer B.Cu) (net 2))
@@
   (segment (start 142.24 66.04) (end 142.24 58.42) (width 0.25) (layer B.Cu) (net 59))
   (segment (start 139.7 58.42) (end 137.16 58.42) (width 0.25) (layer B.Cu) (net 60))
+  (segment (start 118.11 53.975) (end 120.65 53.975) (width 0.25) (layer F.Cu) (net 61))
   (zone (net 7) (net_name GND) (layer B.Cu) (hatch edge 0.508)
     (connect_pads (clearance 0.508))
