File: ILJJ_Mk-V.sch (KiCad schematic (older format))
At the start: 39 parts, among them J1 Conn_02x12, U1 74LS00, U2 74LS00

Commit message: [add] アノテーションとIC電源
ERCも通した
Parts:
- added unit 5 of U1
- added unit 5 of U10
- added unit 5 of U11
- added unit 5 of U2
- added unit 5 of U3
- added unit 5 of U4
- added unit 5 of U5
- added unit 5 of U6
- added unit 5 of U7
- added unit 5 of U8
- added unit 5 of U9
- gave numbers to parts that had none: 9
- renumbered U2 to U7
Connections:
- wire segments 136 -> 156
- no-connect marks 0 -> 6

Commit message: [add] カードエッジ部のフットプリント
Parts:
- J1: footprint (none) -> fplib:5530843-1_edge
- U1, U10, U11, U2, U3, U4, U5, U6, U7, U8, U9: footprint (none) -> Housings_DIP:DIP-14_W7.62mm_LongPads

Commit message: [add] #1 パワーランプ
抵抗のフットプリントこれでいいのかちょっとあやしい
Parts:
- added D1: POWER, LEDs:LED_D3.0mm, symbol Device:LED
- added R1: R, Resistors_ThroughHole:R_Axial_DIN0207_L6.3mm_D2.5mm_P7.62mm_Horizontal, symbol Device:R
Connections:
- wire segments 156 -> 159
Changed lines of the file:
@@
 NoConn ~ 1100 3100
 NoConn ~ 1100 3000
+$Comp
+L power:VCC #PWR07
+U 1 1 5BD9B7F2
+P 950 4000
+F 0 "#PWR07" H 950 3850 50  0001 C CNN
+F 1 "VCC" H 967 4173 50  0000 C CNN
+F 2 "" H 950 4000 50  0001 C CNN
+F 3 "" H 950 4000 50  0001 C CNN
+	1    950  4000
+	1    0    0    -1
+$EndComp
+$Comp
+L Device:R R1
+U 1 1 5BD9BC6D
+P 950 4250
+F 0 "R1" H 1020 4296 50  0000 L CNN
+F 1 "R" H 1020 4205 50  0000 L CNN
+F 2 "Resistors_ThroughHole:R_Axial_DIN0207_L6.3mm_D2.5mm_P7.62mm_Horizontal" V 880 4250 50  0001 C CNN
+F 3 "~" H 950 4250 50  0001 C CNN
+	1    950  4250
+	1    0    0    -1
+$EndComp
+$Comp
+L Device:LED D1
+U 1 1 5BD9BE0F
+P 950 4650
+F 0 "D1" V 988 4532 50  0000 R CNN
+F 1 "POWER" V 897 4532 50  0000 R CNN
+F 2 "LEDs:LED_D3.0mm" H 950 4650 50  0001 C CNN
+F 3 "~" H 950 4650 50  0001 C CNN
+	1    950  4650
+	0    -1   -1   0
+$EndComp
+$Comp
+L power:GND #PWR08
+U 1 1 5BD9BFF2
+P 950 4900
+F 0 "#PWR08" H 950 4650 50  0001 C CNN
+F 1 "GND" H 955 4727 50  0000 C CNN
+F 2 "" H 950 4900 50  0001 C CNN
+F 3 "" H 950 4900 50  0001 C CNN
+	1    950  4900
+	1    0    0    -1
+$EndComp
+Wire Wire Line
+	950  4100 950  4000
+Wire Wire Line
+	950  4400 950  4500
+Wire Wire Line
+	950  4800 950  4900
 $EndSCHEMATC
